File: filter/filter.kicad_pcb (KiCad board)
At the start: 4 copper layers, 36 x 13 mm, 20 parts, among them J1 IN, J2 OUT

Commit message: Prepared for ordering
Other:
- rule via_min_drill: 0.508 -> 0.3
- rule via_min_size: 0.889 -> 0.6
