File: filter/filter.sch (KiCad schematic (older format))
At the start: 20 parts, among them J1 IN, J2 OUT

Commit message: Prepared for ordering
Other:
- note added: "Sever trace to unused filter"
Changed lines of the file:
@@
 LIBS:semi-trans-TI
 LIBS:semi-trans-TIP
-LIBS:semi-trans-Toshiba
 LIBS:silabs
 LIBS:skyworks
@@
 encoding utf-8
 Sheet 1 1
-Title ""
-Date ""
-Rev ""
-Comp ""
-Comment1 ""
+Title "Filter Test PCB"
+Date "2015-02-22"
+Rev "A"
+Comp "WCP52"
+Comment1 "Gain/Phase Analyzer"
 Comment2 ""
 Comment3 ""
@@
 Wire Wire Line
 	6000 4900 6000 4800
+Wire Notes Line
+	2600 2200 3000 2200
+Wire Notes Line
+	3000 2200 3000 2650
+Wire Notes Line
+	3000 2650 2600 2650
+Wire Notes Line
+	2600 2650 2600 2200
+Wire Notes Line
+	8400 2200 8400 2650
+Wire Notes Line
+	8400 2650 8000 2650
+Wire Notes Line
+	8000 2650 8000 2200
+Wire Notes Line
+	8000 2200 8400 2200
+Text Notes 2600 2200 0    60   ~ 0
+Sever trace to unused filter
 $EndSCHEMATC
